Commit message: Imported upstream version '0.4.1' of 'upstream'

File: nextage_description/urdf/NextageOpen.urdf (robot description, URDF)
Before this commit: robot NextageOpen, 16 links, 15 joints
Links:
- removed link WAIST_Link
- added link WAIST, mass 0; collision mesh filename=package://nextage_description/urdf/meshes/WAIST_Link_mesh.d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 scale=1 1 1; visual mesh filename=package://nextage_description/urdf/meshes/WAIST_Link_mesh.d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 scale=1 1 1
Joints:
- joint CHEST_JOINT0: parent WAIST_Link -> WAIST

Commit message: Imported upstream version '0.7.4' of 'upstream'

File: nextage_description/urdf/NextageOpen.urdf (robot description, URDF)
Before this commit: robot NextageOpen, 16 links, 15 joints
Links:
- added link world
- link CHEST_JOINT0_Link: mass 0 -> 3.0
- link WAIST: mass 0 -> 30.0
Joints:
- added joint fixed: type fixed, parent world, child WAIST

Commit message: Imported upstream version '0.7.9' of 'upstream'

File: nextage_description/urdf/NextageOpen.urdf (robot description, URDF)
Before this commit: robot NextageOpen, 17 links, 16 joints
Links:
- removed link world
- link WAIST: mass 30.0 -> 1000
Joints:
- removed joint fixed
- joint LARM_JOINT0: limit lower=-1.53589 upper=1.53589 effort=100 velocity=0.5 -> lower=-1.53589 upper=1.53589 effort=150 velocity=0.5
- joint LARM_JOINT1: limit lower=-2.44346 upper=1.0472 effort=100 velocity=0.5 -> lower=-2.44346 upper=1.0472 effort=200 velocity=0.5
- joint RARM_JOINT0: limit lower=-1.53589 upper=1.53589 effort=100 velocity=0.5 -> lower=-1.53589 upper=1.53589 effort=150 velocity=0.5
- joint RARM_JOINT1: limit lower=-2.44346 upper=1.0472 effort=100 velocity=0.5 -> lower=-2.44346 upper=1.0472 effort=200 velocity=0.5
